File: Hardware/Smart fan controler/Smart Fan Controler.brd (EAGLE design)
At the start: 71.9 x 106.2 mm, 26 parts, among them J1 22-27-2041-04

Commit message: started work on board
Parts:
- removed C4: (no value), rcl:C0805
- removed J3, J7: (no value), SparkFun-Connectors:1X04_LOCK_LONGPADS
- removed R4, R5, R6: (no value), rcl:R0805
- removed U$4: SI3865DDV, DubSat1 Components:TSOP-6
- added C7: (no value), rcl:C0805
- added J4, J8: (no value), Smart fan:MOLEX_FAN_HEADER
- added R13, R14, R15: (no value), rcl:R0805
- added U$8: SI3865DDV, DubSat1 Components:TSOP-6
- J1: value 22-27-2041-04 -> (none); device con-molex:6410-04 -> Smart fan:MOLEX_FAN_HEADER
- J2: device SparkFun-Connectors:1X04_LOCK_LONGPADS -> Smart fan:MOLEX_FAN_HEADER
- moved C5 252.7 mm to (-8.00, 95.5), turned to 270 degrees
- moved R7 251.5 mm to (0.00, 95.6), turned to 90 degrees
- moved R9 251.1 mm to (-1.65, 91.4), turned to 180 degrees
- moved R8 245.0 mm to (-6.22, 91.4)
- moved U$3 234.2 mm to (-18.8, 95.2), turned to 180 degrees
- moved J2 228.9 mm to (-22.9, 102.5)
- moved R1 228.3 mm to (-15.0, 95.5), turned to 90 degrees
- moved R3 223.1 mm to (-16.6, 91.3), turned to 180 degrees
- moved J5 136.8 mm to (-28.7, 64.3), turned to 270 degrees
- moved J6 132.9 mm to (26.5, 33.0), turned to 90 degrees
- moved C1 21.3 mm to (-5.21, 44.1), turned to 270 degrees
- moved C2 17.3 mm to (-0.13, 42.7)
- moved U$1 17.0 mm to (-0.51, 46.2)
- moved C3 17.0 mm to (-23.0, 95.4), turned to 270 degrees
- moved R2 16.5 mm to (-21.2, 91.3)
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Connections:
- removed net N$22: C5.1, J3.2, U$4.P$2, U$4.P$3
- removed net N$23: C3.2, R4.1, U$5.P$6
- new net N$26: C7.1, J8.2, U$8.P$2, U$8.P$3
- new net N$27: C7.2, R14.1, U$8.P$6
- net 0: now also J4.1, J8.1, R13.1, R15.1, R3.1; no longer J3.1, J7.1, R2.1, R5.1, R6.1
- net 12V: now also R14.2, R2.2, U$8.P$4; no longer R3.2, R4.2, U$4.P$4
- net EN1: now also R15.2, U$8.P$5; no longer R9.2, U$4.P$5
- net EN2: now also R9.2; no longer R5.2
- net EN3: now also R3.2; no longer R6.2
- net N$10: now also R7.2, U$5.P$1; no longer C3.1, J7.2, U$5.P$2, U$5.P$3
- net N$11: now also C3.1; no longer C4.1
- net N$19: now also C3.2, R2.1; no longer C4.2, R3.1
- net N$20: now also C5.1, J4.2, U$5.P$2, U$5.P$3; no longer R2.2, U$5.P$1
- net N$21: now also C5.2, R8.1, U$5.P$6; no longer R7.2, U$4.P$1
- net N$25: now also R13.2, U$8.P$1; no longer C5.2, R8.1, U$4.P$6
- net PWM1: now also J8.4; no longer J3.4
- net PWM2: now also J4.4; no longer J7.4
- net SENSE1: now also J8.3; no longer J3.3
- net SENSE2: now also J4.3; no longer J7.3
Routing:
- net 12V: track 0.00 -> 65.4 mm
- net EN3: track 0.00 -> 53.0 mm, vias 0 -> 2
- net EN2: track 0.00 -> 36.9 mm, vias 0 -> 2
- net EN1: track 0.00 -> 20.7 mm, vias 0 -> 2
- net SENSE2: track 0.00 -> 19.8 mm, vias 0 -> 2
- net PWM2: track 0.00 -> 19.1 mm, vias 0 -> 2
- net SENSE3: track 0.00 -> 18.9 mm, vias 0 -> 2
- net PWM3: track 0.00 -> 18.2 mm, vias 0 -> 2
- net N$26: track 0.00 -> 10.6 mm
- net N$20: track 0.00 -> 10.6 mm
- net N$11: track 0.00 -> 10.6 mm
- net 0: track 0.00 -> 10.6 mm
- net N$19: track 0.00 -> 10.2 mm
- net N$27: track 0.00 -> 10.2 mm
- net N$21: track 0.00 -> 10.2 mm
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- added copper zone on layer 16, net 0
