File: Hardware/Smart fan controler/Smart Fan Controler.brd (EAGLE design)
At the start: 93.9 x 106.2 mm, 37 parts

Commit message: Finalized board and made gerber files
Parts:
- moved J3 6.30 mm to (-22.2, 60.1)
- moved C1 6.30 mm to (-14.6, 73.7)
- moved C10 6.30 mm to (49.3, 39.0)
- moved C11 6.30 mm to (42.7, 42.5)
- moved C2 6.30 mm to (-19.3, 75.2)
- moved C3 6.30 mm to (-23.0, 89.1)
- moved C5 6.30 mm to (-8.00, 89.2)
- moved C7 6.30 mm to (6.86, 89.3)
- moved C8 6.30 mm to (49.3, 86.3)
- moved C9 6.30 mm to (42.7, 89.8)
- moved J1 6.30 mm to (27.2, 90.7)
- moved J10 6.30 mm to (37.8, 27.8)
- moved J2 6.30 mm to (-22.9, 96.2)
- moved J4 6.30 mm to (-7.87, 96.3)
- moved J5 6.30 mm to (-30.6, 75.9)
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Other:
- board size 93.9 x 106.2 mm -> 93.9 x 100 mm
