File: Hardware/Smart fan controler/Smart Fan Controler.sch (EAGLE design)
At the start: 26 parts, among them J1 22-27-2041-04

Commit message: started work on board
Parts:
- removed C4: (no value), rcl:C-USC0805
- removed J3, J7: (no value), SparkFun-Connectors:CONN_04LOCK_LONGPADS
- removed R4, R5, R6: (no value), rcl:R-US_R0805
- added C7: (no value), rcl:C-USC0805
- added J4, J8: (no value), Smart fan:CONN_04MOLEX_FAN_HEADER
- added R13, R14, R15: (no value), rcl:R-US_R0805
- J1: value 22-27-2041-04 -> (none); device con-molex:22-27-2041-04 -> Smart fan:CONN_04MOLEX_FAN_HEADER
- J2: device SparkFun-Connectors:CONN_04LOCK_LONGPADS -> Smart fan:CONN_04MOLEX_FAN_HEADER
- renumbered U$4 to U$8
Connections:
- removed net N$22: C5.1, J3.2, U$8.DRAIN1, U$8.DRAIN2
- removed net N$23: C3.2, R4.1, U$5.GATE
- new net N$26: C7.1, J8.2, U$8.DRAIN1, U$8.DRAIN2
- new net N$27: C7.2, R14.1, U$8.GATE
- net 0: now also J1.2, J1.3, J4.1, J8.1, R13.1, R15.1, R3.1; no longer J1-2.S, J1-3.S, J3.1, J7.1, R2.1, R5.1, R6.1
- net 12V: now also J1.1, R14.2, R2.2; no longer J1-1.S, R3.2, R4.2
- net EN1: now also R15.2; no longer R9.2
- net EN2: now also R9.2; no longer R5.2
- net EN3: now also R3.2; no longer R6.2
- net N$10: now also R7.2, U$5.R2; no longer C3.1, J7.2, U$5.DRAIN1, U$5.DRAIN2
- net N$11: now also C3.1; no longer C4.1
- net N$19: now also C3.2, R2.1; no longer C4.2, R3.1
- net N$20: now also C5.1, J4.2, U$5.DRAIN1, U$5.DRAIN2; no longer R2.2, U$5.R2
- net N$21: now also C5.2, R8.1, U$5.GATE; no longer R7.2, U$8.R2
- net N$25: now also R13.2, U$8.R2; no longer C5.2, R8.1, U$8.GATE
- net PWM1: now also J8.4; no longer J3.4
- net PWM2: now also J4.4; no longer J7.4
- net SENSE1: now also J8.3; no longer J3.3
- net SENSE2: now also J4.3; no longer J7.3
Other:
- note removed: "Fan Headers"
- moved on the sheet: C3, C5, R2, R3, R7, R8, R9
