File: Hardware/Smart fan controler/Smart Fan Controler.sch (EAGLE design)
At the start: 26 parts

Commit message: Main board Done
Parts:
- added J3: (no value), SparkFun-Connectors:CONN_05NO_SILK
- added R4, R5: (no value), rcl:R-US_R0805
- added U$4: AIR_QUALITY_SENSOR, Smart fan:AIR_QUALITY_SENSOR
Connections:
- removed net N$12: J6.6
- removed net N$13: J6.5
- removed net N$14: U$1.SCLK
- removed net N$15: U$1.DIN
- removed net N$16: U$1.DOUT
- removed net N$17: J6.4
- removed net N$18: J6.3
- removed net N$6: J5.6
- removed net N$7: J5.5
- removed net N$8: J5.4
- removed net N$9: J5.3
- new net 12VIN: J1.1, R4.2
- new net VOUT: J3.2, U$2.D8
- new net VOUT2: J3.5, U$2.D9
- new net VTH: J3.4, U$2.A5
- net 0: now also J3.3, R5.1
- net 12V: now also R4.1, R5.2; no longer J1.1
- net 5V: now also J3.1, J5.6, J6.6
- net CS1: now also U$2.A4
- net CS2: now also U$2.A6
- net CS3: now also U$2.A7
- net MISO: now also J5.3, J6.3, U$1.DOUT
- net MOSI: now also J5.4, J6.4, U$1.DIN
- net PWM2: no longer U$2.D6
- net PWM3: now also U$2.D6
- net SCLK: now also J5.5, J6.5, U$1.SCLK

Commit message: added breakout board
Parts:
- removed U$6: PCI-E-X1-BOARD, Smart fan:PCI-E-X1-BOARD
- added C10, C11, C8, C9: (no value), rcl:C-USC0805
- added J10, J9: (no value), SparkFun-Connectors:CONN_06LOCK_LONGPADS
- added U$7, U$9: MPL115A1, Smart fan:MPL115A1
Connections:
- new net CS_REMOTE: J10.2, J9.2, U$7.CS, U$9.CS
- new net N$4: C9.1, U$7.CAP
- new net N$5: C11.1, U$9.CAP
- net 0: now also C10.2, C11.2, C8.2, C9.2, J10.1, J9.1, U$7.GND, U$9.GND
- net 5V: now also C10.1, C8.1, J10.6, J9.6, U$7.SHDN, U$7.VDD, U$9.SHDN, U$9.VDD
- net MISO: now also J10.3, J9.3, U$7.DOUT, U$9.DOUT
- net MOSI: now also J10.4, J9.4, U$7.DIN, U$9.DIN
- net SCLK: now also J10.5, J9.5, U$7.SCLK, U$9.SCLK
Other:
- note added: "Breakout Board"
- note added: "PCI-e X1 board shape"
